File: hardware/motion_detector.kicad_pcb (KiCad board)
At the start: 2 copper layers, 45 x 25 mm, 33 parts, among them J1 Debug, P1 CON-SENSOR2, P2 Boot, U1 XMC110024, U3 AM612, U4 DRILL, U5 DRILL, U6 DRILL, U7 DRILL

Commit message: Add 3d information (final)
Parts:
- D2, D3, D4: footprint D1206_INV -> kicad-libraries:D1206_INV
