File: hardware/motion-detector-v2.kicad_pcb (KiCad board)
At the start: 2 copper layers, 45 x 25 mm, 33 parts, among them J1 Debug, P1 CON-SENSOR2, P2 Boot, U1 XMC110024, U3 AM612, U4 DRILL, U5 DRILL, U6 DRILL, U7 DRILL

Commit message: fix status text, add bottom copper masking for sensor
Other:
- board text added: "Status"
- board text removed: "status"
Changed lines of the file:
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@@
-(kicad_pcb (version 20171130) (host pcbnew 5.0.1-33cea8e~67~ubuntu18.04.1)
+(kicad_pcb (version 20171130) (host pcbnew 5.0.2-bee76a0~70~ubuntu18.04.1)
   (general
     (thickness 1.6002)
@@
   (gr_line (start 73.125 37.075) (end 74.175 38.9) (angle 90) (layer Edge.Cuts) (width 0.381))
   (gr_line (start 71.125 38.25) (end 73.125 37.075) (angle 90) (layer Edge.Cuts) (width 0.381))
-  (gr_text status (at 57.3 51.5) (layer F.SilkS)
+  (gr_text Status (at 57.3 51.5) (layer F.SilkS)
     (effects (font (size 0.8 0.8) (thickness 0.15)))
   )
@@
       )
     )
+  )
+  (zone (net 0) (net_name "") (layer Dwgs.User) (hatch edge 0.508)
+    (connect_pads (clearance 0.2))
+    (min_thickness 0.254)
+    (fill yes (arc_segments 16) (thermal_gap 0.508) (thermal_bridge_width 0.508))
+    (polygon
+      (pts
+        (xy 60.9 37.8) (xy 69.9 37.8) (xy 69.9 46.8) (xy 60.9 46.8)
+      )
+    )
